File: hair-02/hair-02.kicad_pcb (KiCad board)
At the start: 2 copper layers, 32 x 32 mm, 33 parts, among them J1 TYPE-C-31-M-12, Q1 2N7002, U1 ESP32-C3-WROOM-02, U2 AP2112K-3.3, U3 TSMP58000

Commit message: hair-02: WIP more routing
Parts:
- removed the D3 at (142.5, 92.7)
- removed the D4 at (160.8, 111.0)
- removed the D5 at (158.2, 99.0)
- removed D6: IR204C-A, LED_THT:LED_D3.0mm
- removed R11: 10R, Resistor_SMD:R_1206_3216Metric
- D1, D2: value IR204C-A -> IR67-21C; footprint LED_THT:LED_D3.0mm -> hair-02:LED_Everlight_IR67-21C
- R10: value 10R -> 33R
- U3: footprint OptoDevice:Vishay_MINICAST-3Pin -> hair-02:Vishay_MINICAST-3Pin-SMD_ReverseMount; moved to B.Cu
- moved R8 35.5 mm to (168.6, 102.2), turned to 0 degrees
- moved R7 33.6 mm to (168.6, 103.9)
- moved C6 32.6 mm to (169.2, 97.3)
- moved C3 19.4 mm to (158.9, 87.2)
- moved R1 19.4 mm to (157.9, 89.8)
- moved R3 19.4 mm to (159.8, 89.8)
- moved U3 17.6 mm to (159.0, 110.8), turned to 0 degrees
- moved R9 15.3 mm to (166.1, 93.3), turned to 0 degrees
- moved R10 13.2 mm to (170.1, 90.2), turned to 90 degrees
- moved RST_SW2 12.3 mm to (152.5, 95.5), turned to 0 degrees
- moved D1 12.3 mm to (148.5, 104.5), turned to 0 degrees
- moved RST_SW1 11.0 mm to (144.5, 95.5)
- moved Q1 11.0 mm to (166.3, 90.0), turned to 90 degrees
- moved D2 7.96 mm to (148.5, 100.5), turned to 180 degrees
- moved C1 4.00 mm to (143.1, 100.3)
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- renumbered D7 to D3, D8 to D4, D9 to D5
Connections:
- R10 pad 1: Net-(Q1-Pad3) -> Net-(D2-Pad1)
- R10 pad 2: Net-(D3-Pad1) -> Net-(Q1-Pad3)
Routing:
- net /~{RESET}: track 12.9 -> 4.24 mm
- net +3V3: track 27.7 -> 20.4 mm
- net /BOOT: track 9.07 -> 3.66 mm
- net Net-(R3-Pad2): track 5.60 -> 1.25 mm
- net GND: track 15.2 -> 17.0 mm
Other:
- board size 32 x 32 mm -> 30 x 24 mm

Commit message: hair-02: Routing done
I'll sleep on it, see if I'm happy with my decisions later
Parts:
- added G***: LOGO, hair:Logo_6mm, F.Cu at (137.5, 98.0)
- moved R8 19.2 mm to (149.4, 103.2), turned to -90 degrees
- moved R10 18.5 mm to (159.0, 105.0), turned to 0 degrees
- moved C6 17.6 mm to (153.4, 105.2), turned to -90 degrees
- moved R7 17.6 mm to (151.0, 103.2), turned to 90 degrees
- moved R3 16.6 mm to (147.8, 101.2)
- moved R1 16.4 mm to (146.2, 101.2)
- moved C3 16.3 mm to (147.2, 98.7)
- moved Q1 16.2 mm to (153.2, 99.5)
- moved R9 15.6 mm to (153.4, 102.5)
- moved D2 10.9 mm to (159.0, 97.5), turned to 0 degrees
- moved D1 10.8 mm to (159.0, 102.0), turned to 180 degrees
Connections:
- D1 pad 2: VBUS -> Net-(D1-Pad2)
- D2 pad 1: Net-(D2-Pad1) -> Net-(Q1-Pad3)
- R10 pad 1: Net-(D2-Pad1) -> VBUS
- R10 pad 2: Net-(Q1-Pad3) -> Net-(D1-Pad2)
- U1 pad 4: /IR_IN -> unconnected-(U1-Pad4)
- U1 pad 6: unconnected-(U1-Pad6) -> /IR_IN
Routing:
- net /IR_IN: track 0.00 -> 37.8 mm, vias 0 -> 2
- net /IR_OUT: track 0.00 -> 11.4 mm, vias 0 -> 1
- net +3V3: track 20.4 -> 30.7 mm
- net VBUS: track 20.7 -> 29.6 mm
- net Net-(C6-Pad1): track 0.00 -> 5.84 mm, vias 0 -> 1
- net Net-(D1-Pad2): track 0.00 -> 5.67 mm
- net Net-(R3-Pad2): track 1.25 -> 6.11 mm
- net Net-(Q1-Pad3): track 0.00 -> 4.69 mm
- net Net-(D1-Pad1): track 0.00 -> 4.50 mm
- net /~{RESET}: track 4.24 -> 8.45 mm
- net GND: track 17.0 -> 20.1 mm, vias 9 -> 11
Other:
- board text added: "hair-02"
- board text added: "icken.ch"

Commit message: hair-02: Add gerbers and interactive BOM
Changed lines of the file:
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@@
     (0 "F.Cu" signal)
     (31 "B.Cu" signal)
-    (32 "B.Adhes" user "B.Adhesive")
-    (33 "F.Adhes" user "F.Adhesive")
     (34 "B.Paste" user)
     (35 "F.Paste" user)
@@
     (40 "Dwgs.User" user "User.Drawings")
     (41 "Cmts.User" user "User.Comments")
-    (42 "Eco1.User" user "User.Eco1")
-    (43 "Eco2.User" user "User.Eco2")
     (44 "Edge.Cuts" user)
     (45 "Margin" user)
@@
     (50 "User.1" user)
     (51 "User.2" user)
-    (52 "User.3" user)
-    (53 "User.4" user)
-    (54 "User.5" user)
-    (55 "User.6" user)
-    (56 "User.7" user)
-    (57 "User.8" user)
-    (58 "User.9" user)
   )
   (setup
@@
       (layerselection 0x00010fc_ffffffff)
       (disableapertmacros false)
-      (usegerberextensions false)
-      (usegerberattributes true)
-      (usegerberadvancedattributes true)
-      (creategerberjobfile true)
+      (usegerberextensions true)
+      (usegerberattributes false)
+      (usegerberadvancedattributes false)
+      (creategerberjobfile false)
       (svguseinch false)
       (svgprecision 6)
@@
       (psa4output false)
       (plotreference true)
-      (plotvalue true)
+      (plotvalue false)
       (plotinvisibletext false)
       (sketchpadsonfab false)
-      (subtractmaskfromsilk false)
+      (subtractmaskfromsilk true)
       (outputformat 1)
       (mirror false)
-      (drillshape 1)
+      (drillshape 0)
       (scaleselection 1)
-      (outputdirectory "")
+      (outputdirectory "gerbers/")
     )
   )
@@
   (net 13 "unconnected-(J1-PadB8)")
   (net 14 "/IR_OUT")
-  (net 15 "Net-(Q1-Pad3)")
+  (net 15 "Net-(D2-Pad1)")
   (net 16 "Net-(R2-Pad2)")
   (net 17 "Net-(R3-Pad2)")
@@
     (fp_line (start 1.6 -0.8) (end 1.6 0.8) (layer "F.Fab") (width 0.1))
     (fp_line (start -1.6 0.8) (end -1.6 -0.8) (layer "F.Fab") (width 0.1))
-    (pad "1" smd roundrect locked (at -1.475 0) (size 1.15 1.8) (layers "F.Cu" "F.Paste" "F.Mask") (roundrect_rratio 0.217391)
+    (pad "1" smd roundrect locked (at -1.475 0) (size 1.15 1.8) (layers "F.Cu" "F.Paste" "F.Mask") (roundrect_rratio 0.2173913043)
       (net 1 "+3V3") (pintype "passive"))
-    (pad "2" smd roundrect locked (at 1.475 0) (size 1.15 1.8) (layers "F.Cu" "F.Paste" "F.Mask") (roundrect_rratio 0.217391)
+    (pad "2" smd roundrect locked (at 1.475 0) (size 1.15 1.8) (layers "F.Cu" "F.Paste" "F.Mask") (roundrect_rratio 0.2173913043)
       (net 2 "GND") (pintype "passive"))
     (model "${KICAD6_3DMODEL_DIR}/Capacitor_SMD.3dshapes/C_1206_3216Metric.wrl"
@@
     (fp_line (start 1.6 0.8) (end -1.6 0.8) (layer "F.Fab") (width 0.1))
     (fp_line (start 1.6 -0.8) (end 1.6 0.8) (layer "F.Fab") (width 0.1))
-    (pad "1" smd roundrect locked (at -1.475 0) (size 1.15 1.8) (layers "F.Cu" "F.Paste" "F.Mask") (roundrect_rratio 0.217391)
+    (pad "1" smd roundrect locked (at -1.475 0) (size 1.15 1.8) (layers "F.Cu" "F.Paste" "F.Mask") (roundrect_rratio 0.2173913043)
       (net 1 "+3V3") (pintype "passive"))
-    (pad "2" smd roundrect locked (at 1.475 0) (size 1.15 1.8) (layers "F.Cu" "F.Paste" "F.Mask") (roundrect_rratio 0.217391)
+    (pad "2" smd roundrect locked (at 1.475 0) (size 1.15 1.8) (layers "F.Cu" "F.Paste" "F.Mask") (roundrect_rratio 0.2173913043)
       (net 2 "GND") (pintype "passive"))
     (model "${KICAD6_3DMODEL_DIR}/Capacitor_SMD.3dshapes/C_1206_3216Metric.wrl"
@@
       (net 2 "GND") (pinfunction "S") (pintype "passive"))
     (pad "3" smd roundrect locked (at 0.9375 0 90) (size 1.475 0.6) (layers "F.Cu" "F.Paste" "F.Mask") (roundrect_rratio 0.25)
-      (net 15 "Net-(Q1-Pad3)") (pinfunction "D") (pintype "passive"))
+      (net 15 "Net-(D2-Pad1)") (pinfunction "D") (pintype "passive"))
     (model "${KICAD6_3DMODEL_DIR}/Package_TO_SOT_SMD.3dshapes/SOT-23.wrl"
       (offset (xyz 0 0 0))
@@
     (fp_line (start -1.6 -1.4) (end 1.6 -1.4) (layer "F.Fab") (width 0.1))
     (pad "1" smd roundrect locked (at -1.5 0) (size 1.5 2.6) (layers "F.Cu" "F.Paste" "F.Mask") (roundrect_rratio 0.25)
-      (net 15 "Net-(Q1-Pad3)") (pinfunction "K") (pintype "passive"))
+      (net 15 "Net-(D2-Pad1)") (pinfunction "K") (pintype "passive"))
     (pad "2" smd roundrect locked (at 1.5 0) (size 1.5 2.6) (layers "F.Cu" "F.Paste" "F.Mask") (roundrect_rratio 0.25)
       (net 6 "Net-(D1-Pad1)") (pinfunction "A") (pintype "passive"))
@@
     (fp_line (start 1.6 0.8) (end -1.6 0.8) (layer "F.Fab") (width 0.1))
     (fp_line (start -1.6 0.8) (end -1.6 -0.8) (layer "F.Fab") (width 0.1))
-    (pad "1" smd roundrect locked (at -1.475 0 270) (size 1.15 1.8) (layers "F.Cu" "F.Paste" "F.Mask") (roundrect_rratio 0.217391)
+    (pad "1" smd roundrect locked (at -1.475 0 270) (size 1.15 1.8) (layers "F.Cu" "F.Paste" "F.Mask") (roundrect_rratio 0.2173913043)
       (net 4 "VBUS") (pintype "passive"))
-    (pad "2" smd roundrect locked (at 1.475 0 270) (size 1.15 1.8) (layers "F.Cu" "F.Paste" "F.Mask") (roundrect_rratio 0.217391)
+    (pad "2" smd roundrect locked (at 1.475 0 270) (size 1.15 1.8) (layers "F.Cu" "F.Paste" "F.Mask") (roundrect_rratio 0.2173913043)
       (net 2 "GND") (pintype "passive"))
     (model "${KICAD6_3DMODEL_DIR}/Capacitor_SMD.3dshapes/C_1206_3216Metric.wrl"
@@
     (fp_line (start -1.6 0.8) (end -1.6 -0.8) (layer "F.Fab") (width 0.1))
     (fp_line (start 1.6 0.8) (end -1.6 0.8) (layer "F.Fab") (width 0.1))
-    (pad "1" smd roundrect locked (at -1.4625 0) (size 1.125 1.75) (layers "F.Cu" "F.Paste" "F.Mask") (roundrect_rratio 0.222222)
+    (pad "1" smd roundrect locked (at -1.4625 0) (size 1.125 1.75) (layers "F.Cu" "F.Paste" "F.Mask") (roundrect_rratio 0.2222222222)
       (net 4 "VBUS") (pintype "passive"))
-    (pad "2" smd roundrect locked (at 1.4625 0) (size 1.125 1.75) (layers "F.Cu" "F.Paste" "F.Mask") (roundrect_rratio 0.222222)
+    (pad "2" smd roundrect locked (at 1.4625 0) (size 1.125 1.75) (layers "F.Cu" "F.Paste" "F.Mask") (roundrect_rratio 0.2222222222)
       (net 7 "Net-(D1-Pad2)") (pintype "passive"))
     (model "${KICAD6_3DMODEL_DIR}/Resistor_SMD.3dshapes/R_1206_3216Metric.wrl"
